Commit message: feat: Update base description

File: packman_description/urdf_xacro/robot.urdf.xacro (robot description, xacro)
@@ -3,9 +3,10 @@
   <xacro:arg name="robot_name" default="" />
   <xacro:include filename="$(find packman_description)/urdf_xacro/robot.gazebo" />
+  <!-- Base -->
   <link name="$(arg robot_name)/base_link">
     <collision name="collision">
-      <origin xyz="0 0 0.08" rpy="0 0 0"/>
+      <origin xyz="0.225 0 0.085" rpy="0 0 0"/>
       <geometry>
-        <box size="0.6 0.4 0.15"/>
+        <box size="0.7 0.5 0.13"/>
       </geometry>
     </collision>
@@ -18,13 +19,27 @@
     </inertial>
     <visual>
-      <origin xyz="0 0 0.08" rpy="0 0 0"/>
+      <origin xyz="0.225 0 0.085" rpy="0 0 0"/>
       <geometry>
-        <box size="0.6 0.4 0.15"/>
+        <box size="0.7 0.5 0.13"/>
+      </geometry>
+    </visual>
+    <visual>
+      <origin xyz="0.035 0 0.17" rpy="0 0 0"/>
+      <geometry>
+        <box size="0.32 0.5 0.04"/>
+      </geometry>
+    </visual>
+    <visual>
+      <origin xyz="0.225 0 0.215" rpy="0 0 0"/>
+      <geometry>
+        <box size="0.7 0.5 0.05"/>
       </geometry>
     </visual>
   </link>
+  </link>
+  <!-- Laser -->
   <joint name="$(arg robot_name)/laser_joint" type="fixed">
     <axis xyz="0 1 0" />
-    <origin xyz="0.31 0 0.075" rpy="0 0 0"/>
+    <origin xyz="0.47 0 0.17" rpy="0 0 0"/>
     <parent link="$(arg robot_name)/base_link"/>
     <child link="$(arg robot_name)/laser_link"/>
@@ -34,5 +49,5 @@
       <origin xyz="0 0 0" rpy="0 0 0"/>
       <geometry>
-        <cylinder length="0.1" radius="0.05"/>
+        <cylinder length="0.05" radius="0.05"/>
       </geometry>
     </visual>

Commit message: feat: Add wheel joints to description

File: packman_description/urdf_xacro/robot.urdf.xacro (robot description, xacro)
@@ -37,4 +37,37 @@
     </visual>
   </link>
+  <!-- Left drive -->
+  <joint name="$(arg robot_name)/left_drive" type="revolute">
+    <parent link="$(arg robot_name)/base_link"/>
+    <child link="$(arg robot_name)/left_wheel_link"/>
+    <origin xyz="0 0.23 0.07525" rpy="${pi / 2} 0 0"/>
+    <axis xyz="0 0 1"/>
+    <limit lower="${-pi}" upper="${pi}" effort="10.0" velocity="30"/>
+    <dynamics damping="0.0" friction="0.0"/>
+  </joint>
+  <link name="$(arg robot_name)/left_wheel_link">
+    <collision>
+      <origin xyz="0 0 0" rpy="0 0 0"/>
+      <geometry>
+        <cylinder radius="0.155" length="0.04"/>
+      </geometry>
+    </collision>
+  </link>
+  <!-- Right drive -->
+  <joint name="$(arg robot_name)/right_drive" type="revolute">
+    <parent link="$(arg robot_name)/base_link"/>
+    <child link="$(arg robot_name)/right_wheel_link"/>
+    <origin xyz="0 -0.23 0.07525" rpy="${pi / 2} 0 0 "/>
+    <axis xyz="0 0 -1"/>
+    <limit lower="${-pi}" upper="${pi}" effort="10.0" velocity="30"/>
+    <dynamics damping="0.0" friction="0.0"/>
+  </joint>
+  <link name="$(arg robot_name)/right_wheel_link">
+    <collision>
+      <origin xyz="0 0 0" rpy="0 0 0"/>
+      <geometry>
+        <cylinder radius="0.155" length="0.04"/>
+      </geometry>
+    </collision>
   </link>
   <!-- Laser -->

Commit message: fix: Fix launch files for the hardware & tune a little

File: packman_description/urdf_xacro/robot.urdf.xacro (robot description, xacro)
@@ -1,8 +1,8 @@
 <?xml version="1.0" encoding="UTF-8"?>
 <robot xmlns:xacro="http://www.ros.org/wiki/xacro" name="robot">
-  <xacro:arg name="robot_name" default="" />
+  <xacro:arg name="robot_prefix" default="" />
   <xacro:include filename="$(find packman_description)/urdf_xacro/robot.gazebo" />
   <!-- Base -->
-  <link name="$(arg robot_name)/base_link">
+  <link name="$(arg robot_prefix)base_link">
     <collision name="collision">
       <origin xyz="0.225 0 0.085" rpy="0 0 0"/>
@@ -38,7 +38,7 @@
   </link>
   <!-- Left drive -->
-  <joint name="$(arg robot_name)/left_drive" type="revolute">
-    <parent link="$(arg robot_name)/base_link"/>
-    <child link="$(arg robot_name)/left_wheel_link"/>
+  <joint name="$(arg robot_prefix)left_wheel" type="revolute">
+    <parent link="$(arg robot_prefix)base_link"/>
+    <child link="$(arg robot_prefix)left_wheel_link"/>
     <origin xyz="0 0.23 0.07525" rpy="${pi / 2} 0 0"/>
     <axis xyz="0 0 1"/>
@@ -46,16 +46,16 @@
     <dynamics damping="0.0" friction="0.0"/>
   </joint>
-  <link name="$(arg robot_name)/left_wheel_link">
+  <link name="$(arg robot_prefix)left_wheel_link">
     <collision>
       <origin xyz="0 0 0" rpy="0 0 0"/>
       <geometry>
-        <cylinder radius="0.155" length="0.04"/>
+        <cylinder radius="0.08" length="0.04"/>
       </geometry>
     </collision>
   </link>
   <!-- Right drive -->
-  <joint name="$(arg robot_name)/right_drive" type="revolute">
-    <parent link="$(arg robot_name)/base_link"/>
-    <child link="$(arg robot_name)/right_wheel_link"/>
+  <joint name="$(arg robot_prefix)right_wheel" type="revolute">
+    <parent link="$(arg robot_prefix)base_link"/>
+    <child link="$(arg robot_prefix)right_wheel_link"/>
     <origin xyz="0 -0.23 0.07525" rpy="${pi / 2} 0 0 "/>
     <axis xyz="0 0 -1"/>
@@ -63,5 +63,5 @@
     <dynamics damping="0.0" friction="0.0"/>
   </joint>
-  <link name="$(arg robot_name)/right_wheel_link">
+  <link name="$(arg robot_prefix)right_wheel_link">
     <collision>
       <origin xyz="0 0 0" rpy="0 0 0"/>
@@ -72,11 +72,11 @@
   </link>
   <!-- Laser -->
-  <joint name="$(arg robot_name)/laser_joint" type="fixed">
+  <joint name="$(arg robot_prefix)laser_joint" type="fixed">
     <axis xyz="0 1 0" />
     <origin xyz="0.47 0 0.17" rpy="0 0 0"/>
-    <parent link="$(arg robot_name)/base_link"/>
-    <child link="$(arg robot_name)/laser_link"/>
+    <parent link="$(arg robot_prefix)base_link"/>
+    <child link="$(arg robot_prefix)laser_link"/>
   </joint>
-  <link name="$(arg robot_name)/laser_link">
+  <link name="$(arg robot_prefix)laser_link">
     <visual>
       <origin xyz="0 0 0" rpy="0 0 0"/>
